File: layouts/default/default.kicad_pcb (KiCad board)
At the start: 2 copper layers, 96.5 x 51.5 mm, 22 parts

Commit message: ready for shipment?
Parts:
- moved C1 195.8 mm to (165.5, 82.0)
- moved C2 195.8 mm to (201.5, 71.5)
- moved C3 195.8 mm to (180.0, 84.5)
- moved C4 195.8 mm to (178.5, 79.5)
- moved C5 195.8 mm to (180.4, 88.0)
- moved KEY1 195.8 mm to (135.9, 100.2)
- moved KEY2 195.8 mm to (158.0, 100.2)
- moved KEY3 195.8 mm to (180.2, 100.2)
- moved KEY4 195.8 mm to (202.4, 100.2)
- moved LED1 195.8 mm to (136.5, 116.5)
- moved LED2 195.8 mm to (158.7, 116.5)
- moved LED3 195.8 mm to (180.8, 116.5)
- moved LED4 195.8 mm to (203.0, 116.5)
- moved R1 195.8 mm to (173.5, 79.5)
- moved R2 195.8 mm to (169.1, 79.5)
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Routing:
- net hid_controller-hv: track 180.9 -> 219.0 mm, vias 4 -> 5
- net DP2: track 0.00 -> 18.3 mm, vias 0 -> 2
- net (no net): track 2.84 -> 0.00 mm
- net A7: track 18.0 -> 19.5 mm
- net gnd: vias 5 -> 27
Other:
- board text added: "Alex Aridgides Work Inc. V0.1.1"

Commit message: update final pcb
Other:
- board text added: "Alex Aridgides Work V0.1.1 atopile {{GITHASH}}"
- board text removed: "Alex Aridgides Work Inc. V0.1.1"
Changed lines of the file:
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@@
 		(layer "Edge.Cuts")
 	)
-	(gr_text "Alex Aridgides\nWork Inc.\nV0.1.1"
-		(at 132 79 0)
-		(layer "F.Cu")
+	(gr_text "Alex Aridgides\nWork\nV0.1.1\natopile\n{{GITHASH}}"
+		(at 132 83.5 0)
+		(layer "F.SilkS")
 		(effects
 			(font
